File: plen2_controlboard.brd (EAGLE design)
At the start: 54 x 43 mm, 120 parts, among them CN1 B5B-ZR, CN2 B5B-ZR, CN3 XH2, CN4 XH2, IC1 24C04SN, J2 3x2M, J3 MYCON2_USB-MINI-B, T1 FDN340P/PMV48XP, T2 PMV48XP, U1 MAX3486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

Commit message: Fix power line
Parts:
- moved U1 0.40 mm to (24.2, 31.9)
- moved C14 0.14 mm to (19.8, 35.3)
- turned CP1 to 270 degrees
Routing:
- net +5V: track 161.0 -> 170.4 mm, vias 8 -> 9
- net GND: track 465.8 -> 457.3 mm
- net RESET: track 68.6 -> 74.9 mm
- net +V1: track 121.6 -> 118.1 mm
- net 3V3: track 31.4 -> 34.3 mm
- net MISO: track 12.0 -> 10.1 mm
- net D1/TX: track 13.4 -> 11.7 mm
- net RS485_B: track 21.0 -> 22.6 mm
- net MOSI: track 15.0 -> 13.8 mm
- net D4*: track 18.3 -> 17.1 mm
- net SCK: track 12.2 -> 11.2 mm
- net SRV12: track 61.0 -> 60.0 mm
- net N$29: track 0.00 -> 0.50 mm
